Commit message: doosan collisions

File: urdf/azure_kinect.urdf.xacro (robot description, xacro)
@@ -6,5 +6,5 @@
 <robot name="azure-kinect" xmlns:xacro="http://www.ros.org/wiki/xacro">
   <xacro:arg name="tf_prefix" default=""/>
-  <material name="black">
+  <!-- <material name="black">
     <color rgba="0. 0. 0. 1" />
   </material>
@@ -17,5 +17,5 @@
   <material name="white">
     <color rgba="0.9 0.9 0.9 1" />
-  </material>
+  </material> -->
   <link name="$(arg tf_prefix)camera_body">
     <visual>
@@ -26,4 +26,9 @@
       <material name="white" />
     </visual>
+    <collision>
+      <geometry>
+          <box size="0.0994 0.0996 0.023" />
+      </geometry>
+    </collision>
   </link>
   <link name="$(arg tf_prefix)camera_base">
@@ -35,4 +40,9 @@
       <material name="grey" />
     </visual>
+    <collision>
+      <geometry>
+          <box size="0.026 0.103 0.039" />
+      </geometry>
+    </collision>
   </link>
   <link name="$(arg tf_prefix)camera_visor">
@@ -44,5 +54,11 @@
       <material name="black" />
     </visual>
+    <collision>
+      <geometry>
+          <box size="0.026 0.101 0.037" />
+      </geometry>
+    </collision>
   </link>
+  <link name="camera_depth"/>
   <joint name="$(arg tf_prefix)camera_base_to_body" type="fixed">
     <parent link="$(arg tf_prefix)camera_base" />
@@ -55,3 +71,89 @@
     <origin xyz="0. 0. 0." rpy="0. 0. 0." />
   </joint>
+  <joint name="$(arg tf_prefix)camera_base_to_depth" type="fixed">
+    <parent link="$(arg tf_prefix)camera_base" />
+    <child link="camera_depth" />
+    <origin xyz="0 0 0 " rpy="-1.57 0 -1.57" />
+  </joint>
+   <!-- camera -->
+  <gazebo reference="camera_base">
+    <sensor type="camera" name="camera">
+      <update_rate>30.0</update_rate>
+      <camera name="head">
+        <horizontal_fov>1.3962634</horizontal_fov>
+        <image>
+          <width>800</width>
+          <height>800</height>
+          <format>R8G8B8</format>
+        </image>
+        <clip>
+          <near>0.02</near>
+          <far>300</far>
+        </clip>
+        <noise>
+          <type>gaussian</type>
+          <!-- Noise is sampled independently per pixel on each frame.
+               That pixel's noise value is added to each of its color
+               channels, which at that point lie in the range [0,1]. -->
+          <mean>0.0</mean>
+          <stddev>0.007</stddev>
+        </noise>
+      </camera>
+      <plugin name="camera_controller" filename="libgazebo_ros_camera.so">
+        <alwaysOn>true</alwaysOn>
+        <updateRate>0.0</updateRate>
+        <cameraName>/camera</cameraName>
+        <imageTopicName>image_raw</imageTopicName>
+        <cameraInfoTopicName>camera_info</cameraInfoTopicName>
+        <frameName>camera_base</frameName>
+        <hackBaseline>0.07</hackBaseline>
+        <distortionK1>0.0</distortionK1>
+        <distortionK2>0.0</distortionK2>
+        <distortionK3>0.0</distortionK3>
+        <distortionT1>0.0</distortionT1>
+        <distortionT2>0.0</distortionT2>
+      </plugin>
+    </sensor>
+  </gazebo>
+  <gazebo reference="camera_base">
+  <sensor name="camera_depth" type="depth">
+    <update_rate>20</update_rate>
+    <camera>
+      <horizontal_fov>1.047198</horizontal_fov>
+      <image>
+        <width>640</width>
+        <height>480</height>
+        <format>R8G8B8</format>
+      </image>
+      <clip>
+        <near>0.02</near>
+        <far>5</far>
+      </clip>
+    </camera>
+    <plugin name="depth_controller" filename="libgazebo_ros_openni_kinect.so">
+      <baseline>0.2</baseline>
+      <alwaysOn>true</alwaysOn>
+      <updateRate>1.0</updateRate>
+      <cameraName>camera_ir</cameraName>
+      <imageTopicName>/camera/depth/image_raw</imageTopicName>
+      <cameraInfoTopicName>/camera/depth/camera_info</cameraInfoTopicName>
+      <depthImageTopicName>/camera/depth/image_raw</depthImageTopicName>
+      <depthImageInfoTopicName>/camera/depth/camera_info</depthImageInfoTopicName>
+      <pointCloudTopicName>/camera/depth/points</pointCloudTopicName>
+      <frameName>camera_depth</frameName>
+      <pointCloudCutoff>0.5</pointCloudCutoff>
+      <pointCloudCutoffMax>3.0</pointCloudCutoffMax>
+      <distortionK1>0.00000001</distortionK1>
+      <distortionK2>0.00000001</distortionK2>
+      <distortionK3>0.00000001</distortionK3>
+      <distortionT1>0.00000001</distortionT1>
+      <distortionT2>0.00000001</distortionT2>
+      <CxPrime>0</CxPrime>
+      <Cx>0</Cx>
+      <Cy>0</Cy>
+      <focalLength>0</focalLength>
+      <hackBaseline>0</hackBaseline>
+    </plugin>
+  </sensor>
+</gazebo>
 </robot>
